File: hardware/pcb/power.kicad_sch (KiCad schematic)
At the start: 52 parts, among them Q1 EPC2305, Q2 EPC2305, U1 LMR36520FADDAR, U2 LMG1210RVRT, U3 LP5907MFX-3.3/NOPB, U6 INA241A2QDGKRQ1

Commit message: Replace legacy passive Specs with verified exact-MPN components
Migrate 51 instances across 20 identities and advance the public library pin to 8a4c96de. Preserve component references, UUIDs, placement, DNP flags, shared package geometry/models and exact pin-to-net connectivity. All ERC findings match baseline; PCB and unrelated components unchanged. Includes per-reference replacement report.
Parts:
- C1, C19, C38: symbol verified:P-00012 -> verified:GRM188R71E104KA01D; IPN P-00012 -> P-00061; IPN_Class Spec -> Part; Manufacturer 1 (none) -> Murata; Manufacturer Part Number 1 (none) -> GRM188R71E104KA01D; Operating Temperature (none) -> -55 to +125 deg C; Package 0603 (1608 Metric) -> 0603; Package Detail (none) -> 0603 (1608 Metric); Rating Conditions (none) -> Nominal 100 nF +/-10%, rated 25 Vdc; X7R temperature charac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; Rev_Creator golanaa -> Steve; Sym_Hash 2542b0e3e5ffcb98 -> c25b734526883d9e; Sym_Version 0.1.1 -> 0.1.0; Tolerance ±10% -> +/-10%; Type SMT -> SMD; Voltage Rating 25 V -> 25 Vdc
- C10, C12, C14, C4, C6, C8: value 2.2 µF -> 2.2uF; symbol verified:P-00015 -> verified:GRM32ER72A225KA35L; Capacitance Measurement Conditions (none) -> Room temperature; 1.0 +/-0.1 kHz; 1.0 +/-0.2 Vrms (p3).; DC Bias Limitation (none) -> Nominal capacitance is not guaranteed at applied DC voltage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; IPN P-00015 -> P-00062; IPN_Class Spec -> Part; Manufacturer 1 (none) -> Murata; Manufacturer Part Number 1 (none) -> GRM32ER72A225KA35L; Maximum Body Height (none) -> 2.70 mm (p2), excluding assembly allowances; Mounting (none) -> Reflow only; evaluate actual PCB lands and solder quantity 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; Operating Temperature (none) -> -55 to +125 C; Package 1210 (3225 Metric) -> 1210; Package Detail (none) -> 1210 (3225 Metric), Murata GRM32E; 3.2 +/-0.3 x 2.5 +/-0.2 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; Packaging (none) -> L: 180 mm reel, W8P4 plastic tape, 1000 pcs/reel; Part Origin (none) -> Exact-MPN migration research from historical P-00015 contex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; Rev_Creator golanaa -> Steve; Sym_Hash 58cc58d737b80d12 -> 60de9d918bb14418; Sym_Version 0.1.1 -> 0.1.0; Temperature Characteristics (none) -> +/-15% from -55 to +125 C, reference 25 C, no DC bias (pp2-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; Tolerance ±10% -> +/-10%; Type SMT -> Multilayer ceramic capacitor (MLCC); Voltage Conditions (none) -> Rated voltage is maximum continuous voltage. With AC superi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; Voltage Rating 100 V -> 100 V DC
- C11, C13, C15, C20, C21, C5, C7, C9: value 22 µF -> 22uF; symbol verified:P-00017 -> verified:GRM32ER71E226KE15L; Capacitance Measurement Conditions (none) -> 22 uF +/-10% measured at room temperature, 120+/-24 Hz, 0.5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; Historical Requirements Comparison (none) -> Nominal 22 uF, 25 V, X7R, +/-10%, 1210 match historical con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; IPN P-00017 -> P-00063; IPN_Class Spec -> Part; Manufacturer 1 (none) -> Murata; Manufacturer Part Number 1 (none) -> GRM32ER71E226KE15L; Operating Temperature (none) -> -55 to +125 C; Package 1210 (3225 Metric) -> 1210; Package Detail (none) -> 1210 (3225 Metric); Part Origin (none) -> New standalone exact-MPN migration from legacy P-00017; no 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; Rev_Creator golanaa -> Steve; Sym_Hash e13dd83282683700 -> 6d2343bae03d1ca1; Sym_Version 0.1.1 -> 0.1.0; Tolerance ±10% -> +/-10%; Voltage Conditions (none) -> 25 V maximum continuous; with AC superimposed on DC, greate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; Voltage Rating 25 V -> 25 VDC
- C16: value 100 nF -> 100nF; symbol verified:P-00016 -> verified:GCM21BR72A104KA37L; Capacitance Measurement Conditions (none) -> 25 C; 1.0 +/-0.1 kHz; 1.0 +/-0.2 Vrms (reference sheet p5); DC Bias Limitations (none) -> Capacitance decreases with applied DC voltage; no numeric e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; IPN P-00016 -> P-00055; IPN_Class Spec -> Part; Manufacturer 1 (none) -> Murata; Manufacturer Part Number 1 (none) -> GCM21BR72A104KA37L; Operating Temperature (none) -> -55 to +125 C; Package 0805 (2012 Metric) -> 0805; Package Detail (none) -> 0805 (2012 Metric); Package Limitations (none) -> Generic lands differ from Murata p27 recommendations; actua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; Packaging (none) -> L: 180 mm reel, 3000 pieces; Part Origin (none) -> Manufacturer reference sheet; shared reviewed managed KiCad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; Rating Conditions (none) -> Applied voltage including transients must remain within rat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; Rev_Creator golanaa -> Steve; Sym_Hash ff9644a485d71a67 -> 7e6233d4181487f4; Sym_Version 0.1.1 -> 0.1.0; Temperature Characteristics (none) -> +/-15% over -55 to +125 C (X7R); not a DC-bias guarantee; Tolerance ±10% -> +/-10%; Voltage Rating 100 V -> 100 VDC
- C17: symbol verified:P-00020 -> verified:GRM21AR72A224KAC5L; IPN P-00020 -> P-00068; IPN_Class Spec -> Part; Manufacturer 1 (none) -> Murata; Manufacturer Part Number 1 (none) -> GRM21AR72A224KAC5L; Operating Temperature (none) -> -55 °C to +125 °C; Package 0805 (2012 Metric) -> 0805; Packaging (none) -> 180 mm embossed tape; Qualification (none) -> General-purpose GRM series; no AEC-Q200 claim.; Rating Conditions (none) -> 100 V DC rated voltage; X7R temperature characteristic. Eff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; Sym_Hash 4cd56f3eb0aee6f7 -> c04f89c501fca84a; Type SMT -> Capacitor; Voltage Rating 100 V -> 100 V DC
- C18, C37: value 1 µF -> 1uF; symbol verified:P-00021 -> verified:GRM21BR71E105KA99L; Capacitance Measurement (none) -> Room temperature; 1 kHz +/-10%; 1.0 +/-0.2 Vrms (spec p.2); DC Bias Limitation (none) -> Effective capacitance decreases with DC bias; exact bias cu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; IPN P-00021 -> P-00047; IPN_Class Spec -> Part; Legacy Comparison (none) -> Nominal 1uF,25V,X7R,+/-10%,0805 agree with legacy context; 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; Manufacturer 1 (none) -> Murata; Manufacturer Part Number 1 (none) -> GRM21BR71E105KA99L; Operating Temperature (none) -> -55 to +125 C; Package 0805 (2012 Metric) -> 0805; Package Detail (none) -> 0805 (2012 Metric); Part Origin (none) -> Exact-MPN symbol created by Steve. Reuses the unchanged rev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; Sym_Hash 1c28230c936da672 -> 0a95b6754c0f7212; Sym_Version 0.1.0 -> 0.1.1; Temperature Characteristic (none) -> +/-15% relative to 25 C over -55 to +125 C; no bias; Tolerance ±10% -> +/-10%; Voltage Rating 25 V -> 25 VDC
- C2, C23, C26: value 2.2 µF -> 2.2 uF; symbol verified:P-00013 -> verified:GRM21BR71A225KA01L; Capacitance (none) -> 2.2 uF; DC Bias (none) -> High dielectric constant capacitance changes with DC bias a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; IPN P-00013 -> P-00054; IPN_Class Spec -> Part; Manufacturer 1 (none) -> Murata; Manufacturer Part Number 1 (none) -> GRM21BR71A225KA01L; Package 0805 (2012 Metric) -> 0805; Package Detail (none) -> 0805 (2012 Metric), 2.0 x 1.25 x 1.25 mm; Rating Conditions (none) -> Room temperature; 1.0±0.1 kHz, 1.0±0.2 Vrms (p3); Rev_Creator golanaa -> Steve; Sym_Hash 6a320f2838449116 -> 2260587002414df2; Sym_Version 0.1.1 -> 0.1.0; Temperature (none) -> -55 to +125 °C; Type SMT -> C; Voltage (none) -> 10 V DC; Voltage Rating 10 V -> 10 V DC
- C22, C24: symbol verified:P-00024 -> verified:12101C475KAT2A; Body Length (none) -> 3.30 ±0.40 mm; Body Width (none) -> 2.50 ±0.30 mm; Capacitance Test Conditions (none) -> 1 kHz ±10%, 1.0 ±0.2 Vrms; after heat treatment where the d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; DC Bias Limitation (none) -> Class II ceramic capacitance varies with applied DC voltage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; IPN P-00024 -> P-00069; IPN_Class Spec -> Part; Manufacturer 1 (none) -> KYOCERA AVX; Manufacturer Part Number 1 (none) -> 12101C475KAT2A; Maximum Height (none) -> 2.79 mm; Operating Temperature Range (none) -> -55 °C to +125 °C; Sym_Hash 5ff5a8df005021d3 -> 417d9fe21fb30c47; Terminal Length (none) -> 0.50 ±0.25 mm; Voltage Rating 100 V -> 100 V DC
- C3: value 220 nF -> 220nF; symbol verified:P-00014 -> verified:GRM188R71C224KA01D; Capacitance Measurement (none) -> Room temperature; 1.0±0.1 kHz, 1.0±0.2 Vrms (datasheet p3); DC Bias Limitation (none) -> High-K capacitance decreases with applied DC voltage; evalu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; IPN P-00014 -> P-00060; IPN_Class Spec -> Part; Manufacturer 1 (none) -> Murata; Manufacturer Part Number 1 (none) -> GRM188R71C224KA01D; Operating Temperature (none) -> -55 to +125 °C; Package 0603 (1608 Metric) -> 0603; Package Detail (none) -> 1608M (0603); Packaging (none) -> D: 180 mm reel, paper tape W8P4, 4000 pcs/reel; Part Origin (none) -> Exact Murata source; reviewed managed generic Capacitor_SMD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; Rev_Creator golanaa -> Steve; Sym_Hash 19a8b23c01c2eba8 -> a408f7bc1e18fd08; Sym_Version 0.1.1 -> 0.1.0; Temperature Characteristics (none) -> ±15% over -55 to +125 °C, reference 25 °C; Voltage Conditions (none) -> Maximum continuous DC 16 V; superimposed AC peak-to-peak or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; Voltage Rating 16 V -> 16 VDC
- R1, R2, R7: value 10 kΩ -> 10k; symbol verified:P-00019 -> verified:RC0402FR-0710KL; IPN P-00019 -> P-00057; IPN_Class Spec -> Part; Manufacturer 1 (none) -> Yageo; Manufacturer Part Number 1 (none) -> RC0402FR-0710KL; Maximum Working Voltage Detail (none) -> 50 V ceiling; actual rated voltage min(sqrt(P*R),50 V) = 25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; Operating Temperature (none) -> -55°C to +155°C; Package 0402 (1005 Metric) -> 0402; Package Detail (none) -> 0402 (1005 Metric); Part Origin (none) -> KiCad Device:R_US symbol graphics; unchanged reviewed manag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; Power Derating (none) -> Full rated power through 70°C ambient; linear derating to z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; Power Rating Conditions (none) -> 70 °C ambient; derate to zero at 155 °C; Power Rating Detail (none) -> 62.5 mW at 70°C ambient; Resistor Technology (none) -> thick film; Sym_Hash 2fe99ffac2e87a7c -> f12e9d89d27ca3f5; Sym_Version 0.1.2 -> 0.1.0; Technology (none) -> Thick film; Terminal Temperature Power Rating (none) -> Not specified in cited RC_L datasheet
- R12: value 2.2 kΩ -> 2.2k; symbol verified:P-00043 -> verified:CRCW20102K20FKEFHP; Additional Power Ratings (none) -> 1.75 W at 105 °C terminal; film ≤155 °C; terminal derating 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; FP_Version 0.1.0 -> 0.1.1; IPN P-00043 -> P-00053; IPN_Class Spec -> Part; Legacy Comparison (none) -> Matches historical 2.2 kohm, 2010, 1%, 100 ppm/K, 1 W P70 a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; Manufacturer 1 (none) -> Vishay; Manufacturer Part Number 1 (none) -> CRCW20102K20FKEFHP; Maximum Working Voltage Detail (none) -> 400 V ACRMS/DC ceiling; additionally limited by sqrt(P*R), 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; Operating Temperature (none) -> -55 °C to +155 °C; Package 2010 (5025 Metric) -> 2010; Part Origin (none) -> Exact-MPN symbol created by Steve. Reuses unchanged managed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; Power Rating Conditions (none) -> 70 °C ambient; film ≤155 °C; derate to zero at 155 °C; Power Rating Detail (none) -> 1.0 W P70 (ambient 70 °C); 1.75 W at terminal 105 °C; Rating Conditions (none) -> Permissible film temperature 155 °C; power rating applies o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; Resistor Technology (none) -> thick film; Sym_Hash 1f1dbe10affec3a1 -> 74e5122f652eb514; Sym_Version 0.1.1 -> 0.1.0; Temperature Coefficient ±100 ppm/°C -> ±100 ppm/K; Type SMT -> Thick Film Resistor
- R14: value 44.2 kΩ -> 44.2k; symbol verified:P-00044 -> verified:RT0402BRD0744K2L; IPN P-00044 -> P-00065; IPN_Class Spec -> Part; Manufacturer 1 (none) -> Yageo; Manufacturer Part Number 1 (none) -> RT0402BRD0744K2L; Operating Temperature (none) -> -55°C to +155°C; Package 0402 (1005 Metric) -> 0402; Package Detail (none) -> 0402 (1005 Metric); Power Derating (none) -> Linear from 62.5 mW at 70°C ambient to 0 W at 155°C; no ter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; Power Rating Conditions (none) -> 70 °C ambient; derate to zero at 155 °C; Power Rating Detail (none) -> 62.5 mW at 70°C ambient; Resistor Technology (none) -> thin film; Sym_Hash f8652e1266a27f5d -> f61990a4f8fa86f5; Sym_Version 0.1.1 -> 0.1.0; Voltage Rating Conditions (none) -> DC or AC rms <= min(50 V, sqrt(P_derated * R))
- R3, R4: value 1 Ω -> 1R; symbol verified:P-00018 -> verified:RC0402FR-071RL; IPN P-00018 -> P-00056; IPN_Class Spec -> Part; Manufacturer 1 (none) -> Yageo; Manufacturer Part Number 1 (none) -> RC0402FR-071RL; Maximum Working Voltage Detail (none) -> 50 V ceiling; limited by sqrt(P*R): 0.25 V at 1 ohm, 62.5 mW; Operating Temperature (none) -> -55 to +155 degC; Package 0402 (1005 Metric) -> 0402; Package Detail (none) -> 0402 (1005 Metric); Power Rating Conditions (none) -> 70 °C ambient; derate to zero at 155 °C; Power Rating Detail (none) -> 62.5 mW at 70 degC ambient; linear derating to 0 W at 155 d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; Resistor Technology (none) -> thick film; Sym_Hash 17252c8c0b1aecc7 -> 239cf666f5555759; Sym_Version 0.1.2 -> 0.1.0; Temperature Coefficient Detail (none) -> +/-200 ppm/degC (1 ohm <= R <= 10 ohm); Terminal Temperature Power Rating (none) -> Not specified (ambient rating only); Tolerance ±1% -> +/-1%
- R5: value 100 kΩ -> 100k; symbol verified:P-00022 -> verified:RC0402FR-07100KL; Dielectric Withstanding Voltage (none) -> 100 V; IPN P-00022 -> P-00058; IPN_Class Spec -> Part; Lifecycle (none) -> Unverified; Manufacturer 1 (none) -> Yageo; Manufacturer Part Number 1 (none) -> RC0402FR-07100KL; Maximum Overload Voltage (none) -> 100 V (short-time overload, not continuous working voltage); Maximum Working Voltage Detail (none) -> 50 V; continuous voltage limited to min(sqrt(P_derated * R)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; Migration Comparison (none) -> Historical numerical targets agree with this exact MPN unde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; Model Limitations (none) -> Measured catalog STEP bounding box 1.00 x 0.50 x 0.35 mm, z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; Mounting Type (none) -> SMD; Operating Temperature (none) -> -55 °C to +155 °C; Package 0402 (1005 Metric) -> 0402; Package Detail (none) -> 0402 (1005 Metric); Power Rating Conditions (none) -> 70 °C ambient; derate to zero at 155 °C; Power Rating Conditions Detail (none) -> 1/16 W at 70 °C ambient; linear derating to 0 W at 155 °C a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; Power Rating Detail (none) -> 0.0625 W; Rating Source (none) -> Yageo RC_L V14 pp2,5,7; Resistance (none) -> 100 kOhm; Resistor Technology (none) -> thick film; Resistor Technology Detail (none) -> Thick film; Sym_Hash 0619541f735b2311 -> a1e8c37e7bc93350; Type SMT -> Resistor; Voltage Rating (none) -> 50 V
- R6: value 24.9 kΩ -> 24.9k; symbol verified:P-00023 -> verified:RC0402FR-0724K9L; IPN P-00023 -> P-00059; IPN_Class Spec -> Part; Manufacturer 1 (none) -> Yageo; Manufacturer Part Number 1 (none) -> RC0402FR-0724K9L; Operating Temperature (none) -> -55 to +155 C; Package 0402 (1005 Metric) -> 0402; Package Detail (none) -> 0402 (1005 Metric), Yageo RC0402; Part Origin (none) -> Manufacturer RC_L evidence; existing reviewed managed R_040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; Power (none) -> 62.5 mW at 70 C ambient; derates to 0 at 155 C; Power Rating Conditions (none) -> 70 °C ambient; derate to zero at 155 °C; Resistance (none) -> 24.9k; Resistor Technology (none) -> thick film; Sym_Hash 6aa389074e380ef5 -> f776139d9b6a89ff; Temperature Coefficient ±100 ppm/°C -> +/-100 ppm/C; Tolerance ±1% -> +/-1%; Type SMT -> Resistor; Voltage (none) -> 50 V maximum; continuous min(50 V, sqrt(P*R))
- R8: value 402 kΩ -> 402k; symbol verified:P-00033 -> verified:TNPW0805402KBEEA; Additional Power Ratings (none) -> 220/260 mW at 70 °C ambient with film ≤155/175 °C (power/ad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; IPN P-00033 -> P-00049; IPN_Class Spec -> Part; Legacy Comparison (none) -> Historical 402 kohm, 0.1%, 25 ppm/C and 0805 match. 150 V r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; Manufacturer 1 (none) -> Vishay Dale; Manufacturer Part Number 1 (none) -> TNPW0805402KBEEA; Maximum Working Voltage 100 V -> 150 V; Maximum Working Voltage Detail (none) -> 150 V AC RMS/DC; also limited by sqrt(P*R); Package 0805 (2012 Metric) -> 0805; Package Detail (none) -> 0805 (2012 Metric); Part Origin (none) -> Exact-MPN symbol created by Steve. Reuses the unchanged rev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; Power Rating 125 mW -> 140 mW; Power Rating Conditions (none) -> 70 °C ambient, general mode; film ≤125 °C; derating applies; Power Rating Detail (none) -> P70 ambient: 0.140 W / 0.220 W / 0.260 W for 125 / 155 / 17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; Rating Conditions (none) -> Derate ambient power linearly above 70 C to zero at selecte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; Resistor Technology (none) -> thin film; Sym_Hash 22eb248036c0adbd -> ecedf9a3ef721d87; Temperature Coefficient Detail (none) -> +/-25 ppm/K; Tolerance ±0.1% -> +/-0.1%; Type SMT -> Thin film resistor
- R9: value 100 kΩ -> 100k; symbol verified:P-00034 -> verified:TNPW0805100KBEEA; Additional Power Ratings (none) -> 220/260 mW at 70 °C ambient with film ≤155/175 °C (power/ad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; Historical Requirement Comparison (none) -> Historical 100 kohm, +/-0.1%, +/-25 ppm/degC and 0805 match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; IPN P-00034 -> P-00050; IPN_Class Spec -> Part; Manufacturer 1 (none) -> Vishay Dale; Manufacturer Part Number 1 (none) -> TNPW0805100KBEEA; Maximum Working Voltage 100 V -> 150 V; Operating Temperature (none) -> -55 to +175 degC advanced; general upper limit +125 degC, p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; Ordering (none) -> TNPW0805 / 100K / B / E / EA; EA lead-free paper tape, 5000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; Package 0805 (2012 Metric) -> 0805; Package Detail (none) -> 0805 (2012 Metric); nominal 2.00 x 1.25 x 0.45 mm; Part Origin (none) -> Exact-MPN symbol created by Steve. Reuses the unchanged rev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; Power Rating 125 mW -> 140 mW; Power Rating Conditions (none) -> 70 °C ambient, general mode; film ≤125 °C; derating applies; Power Rating Conditions Detail (none) -> Permissible film temperatures: general 125 degC, power 155 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; Power Rating Detail (none) -> P70: 0.140 W general / 0.220 W power / 0.260 W advanced ope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; Resistance (none) -> 100 kohm; Resistor Technology (none) -> thin film; Sym_Hash 735a21acf441f303 -> 7af933fb13accaf4; Temperature Coefficient ±25 ppm/°C -> +/-25 ppm/K; Terminal Temperature Power Rating (none) -> 0.75 W at terminal part temperature 105 degC; application t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; Tolerance ±0.1% -> +/-0.1%; Voltage Rating (none) -> 150 V maximum operating voltage, AC RMS or DC; power and vo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

Commit message: Update precision current-sense circuit and pin published OCPM library
Parts:
- removed R10: 5 mΩ, verified:SEWF3920D5L00P9_PCB, symbol verified:SEWF3920D5L00P9
- added C39, C40, C41: 100 nF, verified:C_0603_1608Metric, symbol verified:GRM188R71E104KA01D
- added R10: 5 mΩ, verified:R_2512_6332Metric, symbol verified:PK2512FKE570R005L
- added R15: 40 kΩ, verified:R_0402_1005Metric, symbol verified:RNCF0402BTE40K0
- added R16: 1 kΩ, verified:R_0402_1005Metric, symbol verified:RC0402FR-071KL
- added R17: 10 kΩ, verified:R_0402_1005Metric, symbol verified:RNCF0402BTE10K0
- added U5: OPA333AIDBVR, verified:OPA333AIDBVR_PCB, symbol verified:OPA333AIDBVR
Connections:
- net 2V5: now also R15.1
- net 3V3: now also C37.1, C38.1, U6.6 (VS), C39.1, U5.5 (V+)
- net 5V0: no longer C37.1, C38.1, U6.6 (VS)
- net GND: now also C39.2, C40.2, C41.2, R17.2, U5.2 (V-)
- net IOUT_SENSE: now also C41.1, R16.2; no longer U6.5 (OUT)
- net MPPT_BUS: now also R10.2
- net at U6.3 (REF2): now also U6.7 (REF1), U5.1, U5.4 (-)
- net at L1.2, U6.8 (IN+): now also R10.1
- new net: R16.1, U6.5 (OUT)
- new net: C40.1, R15.2, R17.1, U5.3 (+)
Other:
- note added: "0.5V Offset"
- note added: "need higher voltage diodes?"
- moved on the sheet: C11, C13, C15, C37, C38, C5, C7, C9, U6
